File: ryloo.kicad_pcb (KiCad board)
At the start: 2 copper layers, 19.7 x 13.9 mm, 6 parts, among them J1 HRO-TYPE-C-31-M-12, J2 Conn_01x04

Commit message: Upload rev2 files
Parts:
- added F1: Polyfuse, Keeb_components:F_0805, F.Cu at (6.20, -2.40)
- added U1: USBLC6-2SC6, Keeb_components:USBLC6-2SC6, F.Cu at (9.95, -3.65)
- moved R2 12.4 mm to (3.95, -2.40)
- moved J2 6.27 mm to (15.7, -0.90)
- moved R1 1.81 mm to (1.70, -2.40)
Connections:
- J1 pad 11: VCC -> VBUS
- J1 pad 2: VCC -> VBUS
- J1 pad 3: Net-(J1-Pad3) -> (no net)
- J1 pad 5: D- -> Net-(J1-Pad5)
- J1 pad 6: D+ -> Net-(J1-Pad6)
- J1 pad 7: D- -> Net-(J1-Pad5)
- J1 pad 8: D+ -> Net-(J1-Pad6)
- J1 pad 9: Net-(J1-Pad9) -> (no net)
Routing:
- net GND: track 54.4 -> 13.9 mm, vias 2 -> 3
- net VBUS: track 0.00 -> 23.1 mm, vias 0 -> 4
- net VCC: track 15.9 -> 8.43 mm
- net Net-(J1-Pad5): track 0.00 -> 6.27 mm
- net D-: track 13.1 -> 6.93 mm, vias 2 -> 0
- net Net-(J1-Pad6): track 0.00 -> 6.19 mm
- net D+: track 5.77 -> 10.6 mm
- net Net-(J1-Pad4): track 9.91 -> 11.1 mm
- added copper zone on B.Cu, net GND
- added copper zone on F.Cu, net GND
Other:
- board size 19.7 x 13.9 mm -> 21.2 x 16.1 mm
- board text added: "rev2"
- board text removed: "rev1"

Commit message: QOL improvements
Parts:
- J1: footprint Keeb_components:HRO-TYPE-C-31-M-12 -> Keeb_components:CONN_HRO-TYPE-C-31-M-12
- J2: footprint Keeb_components:JST_SH_SM04B-SRSS-TB_1x04-1MP_P1.00mm_Horizontal -> Keeb_components:CONN_JST_SH_SM04B-SRSS-TB_1x04-1MP_P1.00mm_Horizontal
- U1: footprint Keeb_components:USBLC6-2SC6 -> Keeb_components:PACKAGE_SOT-23-6
- turned J1 to 0 degrees
- turned U1 to 90 degrees
Connections:
- J1 pad 3: (no net) -> unconnected-(J1-Pad3)
- J1 pad 9: (no net) -> unconnected-(J1-Pad9)
Routing:
- net VBUS: track 23.1 -> 21.2 mm
Other:
- board text added: "rev2.1"
- board text removed: "rev2"
