File: ryloo.kicad_sch (KiCad schematic)
At the start: 4 parts, among them J1 HRO-TYPE-C-31-M-12, J2 Conn_01x04

Commit message: Upload rev2 files
Parts:
- added F1: Polyfuse, Keeb_components:F_0805, symbol Device:Polyfuse
- added U1: USBLC6-2SC6, Keeb_components:USBLC6-2SC6, symbol keyboard_parts:USBLC6-2SC6
Connections:
- net D+: now also U1.4 (I/O2); no longer J1.6 (DP1), J1.8 (DP2)
- net D-: now also U1.6 (I/O1); no longer J1.5 (DN2), J1.7 (DN1)
- net GND: now also U1.2 (GND)
- net VCC: now also F1.2; no longer J1.11 (VBUS), J1.2 (VBUS)
- new net: J1.5 (DN2), J1.7 (DN1), U1.1 (I/O1)
- new net: J1.6 (DP1), J1.8 (DP2), U1.3 (I/O2)
- new net VBUS: F1.1, J1.11 (VBUS), J1.2 (VBUS), U1.5 (VBUS)
Other:
- moved on the sheet: J2

Commit message: QOL improvements
Parts:
- J1: footprint Keeb_components:HRO-TYPE-C-31-M-12 -> Keeb_components:CONN_HRO-TYPE-C-31-M-12
- J2: footprint Keeb_components:JST_SH_SM04B-SRSS-TB_1x04-1MP_P1.00mm_Horizontal -> Keeb_components:CONN_JST_SH_SM04B-SRSS-TB_1x04-1MP_P1.00mm_Horizontal
- U1: footprint Keeb_components:USBLC6-2SC6 -> Keeb_components:PACKAGE_SOT-23-6
Changed lines of the file:
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@@
       (effects (font (size 1.524 1.524)))
     )
-    (property "Footprint" "Keeb_components:HRO-TYPE-C-31-M-12" (id 2) (at 58.42 66.04 0)
+    (property "Footprint" "Keeb_components:CONN_HRO-TYPE-C-31-M-12" (id 2) (at 58.42 66.04 0)
       (effects (font (size 1.524 1.524)) hide)
     )
@@
       (effects (font (size 1.27 1.27)) (justify left))
     )
-    (property "Footprint" "Keeb_components:JST_SH_SM04B-SRSS-TB_1x04-1MP_P1.00mm_Horizontal" (id 2) (at 158.75 90.805 0)
+    (property "Footprint" "Keeb_components:CONN_JST_SH_SM04B-SRSS-TB_1x04-1MP_P1.00mm_Horizontal" (id 2) (at 158.75 90.805 0)
       (effects (font (size 1.27 1.27)) hide)
     )
@@
     (property "Reference" "U1" (id 0) (at 118.11 72.39 0))
     (property "Value" "USBLC6-2SC6" (id 1) (at 118.11 69.85 0))
-    (property "Footprint" "Keeb_components:USBLC6-2SC6" (id 2) (at 110.49 71.12 0)
+    (property "Footprint" "Keeb_components:PACKAGE_SOT-23-6" (id 2) (at 110.49 71.12 0)
       (effects (font (size 1.27 1.27)) (justify left) hide)
     )
@@
     )
     (path "/00000000-0000-0000-0000-00005c91af59"
-      (reference "J1") (unit 1) (value "HRO-TYPE-C-31-M-12") (footprint "Keeb_components:HRO-TYPE-C-31-M-12")
+      (reference "J1") (unit 1) (value "HRO-TYPE-C-31-M-12") (footprint "Keeb_components:CONN_HRO-TYPE-C-31-M-12")
     )
     (path "/00000000-0000-0000-0000-00005c91afcb"
-      (reference "J2") (unit 1) (value "Conn_01x04") (footprint "Keeb_components:JST_SH_SM04B-SRSS-TB_1x04-1MP_P1.00mm_Horizontal")
+      (reference "J2") (unit 1) (value "Conn_01x04") (footprint "Keeb_components:CONN_JST_SH_SM04B-SRSS-TB_1x04-1MP_P1.00mm_Horizontal")
     )
     (path "/00000000-0000-0000-0000-00005c91b042"
@@
     )
     (path "/0c6553f1-2edc-42e5-b228-c8f88411feef"
-      (reference "U1") (unit 1) (value "USBLC6-2SC6") (footprint "Keeb_components:USBLC6-2SC6")
-    )
-  )
+      (reference "U1") (unit 1) (value "USBLC6-2SC6") (footprint "Keeb_components:PACKAGE_SOT-23-6")
+    )
+  )
